File: KiCAD files/TDS1.kicad_sch (KiCad schematic)
At the start: 16 parts, among them J1 Conn_01x02_Pin, J2 Conn_01x02_Pin, J3 Conn_01x02_Pin, U1 TL072

Commit message: pcb and schematic
Parts:
- C1, C2, C3, C4: value 10uF -> 10µF
- R1, R3, R4: value 10k -> 10kΩ
- R2, RV1, RV2: value 100k -> 100kΩ
- R5, R6: value 1k -> 1kΩ
Connections:
- net GND: no longer RV2.1
- net at C1.1, R6.1, RV2.2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: now also RV2.1
Changed lines of the file:
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@@
+	)
+	(junction
+		(at 156.21 111.76)
+		(diameter 0)
+		(color 0 0 0 0)
+	)
+	(junction
+		(at 161.29 111.76)
+		(diameter 0)
+		(color 0 0 0 0)
 	)
 	(junction
@@
 	)
 	(junction
-		(at 161.29 118.11)
-		(diameter 0)
-		(color 0 0 0 0)
-	)
-	(junction
 		(at 137.16 111.76)
 		(diameter 0)
@@
 	(wire
 		(pts
+			(xy 154.94 111.76) (xy 156.21 111.76)
+		)
+		(stroke
+			(width 0)
+			(type default)
+		)
+	)
+	(wire
+		(pts
 			(xy 184.15 87.63) (xy 184.15 77.47)
 		)
@@
 	(wire
 		(pts
+			(xy 151.13 116.84) (xy 156.21 116.84)
+		)
+		(stroke
+			(width 0)
+			(type default)
+		)
+	)
+	(wire
+		(pts
 			(xy 167.64 80.01) (xy 165.1 80.01)
 		)
@@
 	(wire
 		(pts
-			(xy 151.13 115.57) (xy 151.13 118.11)
-		)
-		(stroke
-			(width 0)
-			(type default)
-		)
-	)
-	(wire
-		(pts
 			(xy 137.16 111.76) (xy 147.32 111.76)
 		)
@@
 	(wire
 		(pts
-			(xy 161.29 118.11) (xy 161.29 102.87)
+			(xy 161.29 118.11) (xy 161.29 111.76)
 		)
 		(stroke
@@
 	(wire
 		(pts
+			(xy 161.29 111.76) (xy 161.29 102.87)
+		)
+		(stroke
+			(width 0)
+			(type default)
+		)
+	)
+	(wire
+		(pts
 			(xy 109.22 100.33) (xy 114.3 100.33)
 		)
@@
 	(wire
 		(pts
+			(xy 156.21 111.76) (xy 161.29 111.76)
+		)
+		(stroke
+			(width 0)
+			(type default)
+		)
+	)
+	(wire
+		(pts
 			(xy 127 127) (xy 123.19 127)
 		)
@@
 	(wire
 		(pts
-			(xy 151.13 118.11) (xy 161.29 118.11)
+			(xy 151.13 116.84) (xy 151.13 115.57)
 		)
 		(stroke
@@
 		(pts
 			(xy 127 127) (xy 127 128.27)
+		)
+		(stroke
+			(width 0)
+			(type default)
+		)
+	)
+	(wire
+		(pts
+			(xy 156.21 116.84) (xy 156.21 111.76)
 		)
 		(stroke
@@
 			)
 		)
-		(property "Value" "100k"
+		(property "Value" "100kΩ"
 			(at 151.13 109.474 90)
 			(effects
@@
 			)
 		)
-		(property "Value" "10k"
-			(at 102.616 117.348 90)
+		(property "Value" "10kΩ"
+			(at 102.616 118.11 90)
 			(effects
 				(font
@@
 			)
 		)
-		(property "Value" "10uF"
+		(property "Value" "10µF"
 			(at 130.556 118.11 90)
 			(effects
@@
 			)
 		)
-		(property "Value" "10uF"
+		(property "Value" "10µF"
 			(at 112.776 117.856 90)
 			(effects
@@
 			)
 		)
-		(property "Value" "10k"
-			(at 171.196 117.348 90)
+		(property "Value" "10kΩ"
+			(at 171.196 118.11 90)
 			(effects
 				(font
@@
 		(on_board yes)
 		(dnp no)
-		(fields_autoplaced yes)
 		(property "Reference" "R6"
-			(at 163.83 120.6499 0)
+			(at 161.29 123.19 90)
 			(effects
 				(font
@@
 			)
 		)
-		(property "Value" "1k"
-			(at 163.83 123.1899 0)
+		(property "Value" "1kΩ"
+			(at 163.576 123.952 90)
 			(effects
 				(font
@@
 			)
 		)
-		(property "Value" "10k"
-			(at 102.616 85.598 90)
+		(property "Value" "10kΩ"
+			(at 102.616 86.36 90)
 			(effects
 				(font
@@
 			)
 		)
-		(property "Value" "10uF"
+		(property "Value" "10µF"
 			(at 140.716 125.73 90)
 			(effects
@@
 			)
 		)
-		(property "Value" "10uF"
+		(property "Value" "10µF"
 			(at 165.1 106.426 90)
 			(effects
@@
 			)
 		)
-		(property "Value" "100k"
-			(at 179.324 113.03 90)
+		(property "Value" "100kΩ"
+			(at 179.07 112.268 90)
 			(effects
 				(font
@@
 				(path "/5a6efc3c-4e23-4ab1-9ce7-0fd5ce7a22d7"
 					(reference "RV1")
-					(unit 1)
-				)
-			)
-		)
-	)
-	(symbol
-		(lib_id "power:GND")
-		(at 154.94 111.76 90)
-		(unit 1)
-		(exclude_from_sim no)
-		(in_bom yes)
-		(on_board yes)
-		(dnp no)
-		(property "Reference" "#PWR05"
-			(at 161.29 111.76 0)
-			(effects
-				(font
-					(size 1.27 1.27)
-				)
-				(hide yes)
-			)
-		)
-		(property "Value" "GND"
-			(at 156.972 113.284 90)
-			(effects
-				(font
-					(size 1.27 1.27)
-				)
-				(justify right)
-			)
-		)
-		(property "Footprint" ""
-			(at 154.94 111.76 0)
-			(effects
-				(font
-					(size 1.27 1.27)
-				)
-				(hide yes)
-			)
-		)
-		(property "Datasheet" ""
-			(at 154.94 111.76 0)
-			(effects
-				(font
-					(size 1.27 1.27)
-				)
-				(hide yes)
-			)
-		)
-		(property "Description" "Power symbol creates a global label with name \"GND\" , ground"
-			(at 154.94 111.76 0)
-			(effects
-				(font
-					(size 1.27 1.27)
-				)
-				(hide yes)
-			)
-		)
-		(pin "1"
-		)
-		(instances
-			(project "TDS1"
-				(path "/5a6efc3c-4e23-4ab1-9ce7-0fd5ce7a22d7"
-					(reference "#PWR05")
 					(unit 1)
 				)
@@
 			)
 		)
-		(property "Value" "1k"
-			(at 139.446 116.586 90)
+		(property "Value" "1kΩ"
+			(at 139.446 117.602 90)
 			(effects
 				(font
@@
 			)
 		)
-		(property "Value" "100k"
+		(property "Value" "100kΩ"
 			(at 118.11 102.616 90)
 			(effects
